File: pcb/pcb.kicad_pcb (KiCad board)
At the start: 2 copper layers, 76.8 x 75 mm, 38 parts, among them J1 Conn_01x04, SW1 SW_Push, SW10 SW_Push, SW11 SW_Push, SW12 SW_Push, SW2 SW_Push, SW3 SW_Push, SW4 SW_Push, SW5 SW_Push, SW6 SW_Push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

Commit message: Finished PCB
Parts:
- moved D10 2.59 mm to (192.4, 113.5)
- moved D11 2.59 mm to (211.4, 113.5)
- moved D12 2.59 mm to (230.5, 113.5)
- moved D5 2.59 mm to (173.3, 94.5)
- moved D6 2.59 mm to (192.4, 94.5)
- moved D7 2.59 mm to (211.4, 94.5)
- moved D8 2.59 mm to (230.5, 94.5)
- moved D9 2.59 mm to (173.3, 113.5)
Routing:
- net +5V: track 0.00 -> 375.8 mm, vias 0 -> 25
- net R3: track 0.00 -> 147.1 mm, vias 0 -> 2
- net R2: track 0.00 -> 112.8 mm, vias 0 -> 1
- net R1: track 0.00 -> 110.2 mm
- net C1: track 0.00 -> 95.8 mm, vias 0 -> 1
- net C4: track 0.00 -> 78.1 mm, vias 0 -> 1
- net SCL: track 0.00 -> 76.6 mm
- net C2: track 0.00 -> 63.6 mm, vias 0 -> 1
- net SDA: track 0.00 -> 62.0 mm
- net C3: track 0.00 -> 55.1 mm, vias 0 -> 3
- net LED_IN: track 0.00 -> 52.4 mm, vias 0 -> 1
- net Net-(D20-DOUT): track 0.00 -> 40.3 mm, vias 0 -> 2
- net Net-(D16-DOUT): track 0.00 -> 36.1 mm, vias 0 -> 2
- net Net-(D18-DOUT): track 0.00 -> 30.8 mm, vias 0 -> 2
- net Net-(D17-DOUT): track 0.00 -> 30.5 mm
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- added copper zone on B.Cu, net GND
- added copper zone on F.Cu, net GND
Other:
- outline, holes or cut-outs redrawn
